File: project2/project2.kicad_pcb (KiCad board)
At the start: 2 copper layers, 100.7 x 64 mm, 22 parts, among them U1 W29C020, U2 W29C020, U3 74LS32, U4 74LS04, U5 74LS670, U6 74LS139, U7 74LS670

Commit message: :a
Signed-off-by: ykp74 <ykp7409@gmail.com>
Routing:
- net GND: vias 147 -> 157
Changed lines of the file:
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@@
     (property "ki_keywords" "R res resistor")
     (attr through_hole)
-    (fp_text reference "R1" (at 5.08 -2.37) (layer "F.SilkS")
+    (fp_text reference "R1" (at 0.067294 2.052101) (layer "F.SilkS")
         (effects (font (size 1 1) (thickness 0.15)))
     )
@@
     (property "ki_keywords" "R res resistor")
     (attr through_hole)
-    (fp_text reference "R4" (at 0.459187 1.811532) (layer "F.SilkS")
+    (fp_text reference "R4" (at 0.05053 1.942405) (layer "F.SilkS")
         (effects (font (size 1 1) (thickness 0.15)))
     )
@@
   (via (at 124.46 86.36) (size 0.8) (drill 0.4) (layers "F.Cu" "B.Cu") (free) (net 6))
   (via (at 104.14 78.74) (size 0.8) (drill 0.4) (layers "F.Cu" "B.Cu") (free) (net 6))
+  (via (at 185.42 78.74) (size 0.8) (drill 0.4) (layers "F.Cu" "B.Cu") (free) (net 6))
   (via (at 157.48 86.36) (size 0.8) (drill 0.4) (layers "F.Cu" "B.Cu") (free) (net 6))
   (via (at 96.52 81.28) (size 0.8) (drill 0.4) (layers "F.Cu" "B.Cu") (free) (net 6))
   (via (at 160.16053 120.632128) (size 0.8) (drill 0.4) (layers "F.Cu" "B.Cu") (free) (net 6))
+  (via (at 185.42 83.82) (size 0.8) (drill 0.4) (layers "F.Cu" "B.Cu") (free) (net 6))
   (via (at 124.46 114.3) (size 0.8) (drill 0.4) (layers "F.Cu" "B.Cu") (free) (net 6))
   (via (at 177.8 119.38) (size 0.8) (drill 0.4) (layers "F.Cu" "B.Cu") (free) (net 6))
@@
   (via (at 93.98 93.98) (size 0.8) (drill 0.4) (layers "F.Cu" "B.Cu") (free) (net 6))
   (via (at 142.200543 75.611643) (size 0.8) (drill 0.4) (layers "F.Cu" "B.Cu") (free) (net 6))
+  (via (at 139.7 73.66) (size 0.8) (drill 0.4) (layers "F.Cu" "B.Cu") (free) (net 6))
   (via (at 96.52 78.74) (size 0.8) (drill 0.4) (layers "F.Cu" "B.Cu") (free) (net 6))
   (via (at 182.88 86.36) (size 0.8) (drill 0.4) (layers "F.Cu" "B.Cu") (free) (net 6))
   (via (at 148.220201 115.67709) (size 0.8) (drill 0.4) (layers "F.Cu" "B.Cu") (free) (net 6))
+  (via (at 185.42 116.84) (size 0.8) (drill 0.4) (layers "F.Cu" "B.Cu") (free) (net 6))
   (via (at 135.868762 113.753054) (size 0.8) (drill 0.4) (layers "F.Cu" "B.Cu") (free) (net 6))
   (via (at 170.18 106.68) (size 0.8) (drill 0.4) (layers "F.Cu" "B.Cu") (free) (net 6))
@@
   (via (at 101.6 119.38) (size 0.8) (drill 0.4) (layers "F.Cu" "B.Cu") (free) (net 6))
   (via (at 180.34 119.38) (size 0.8) (drill 0.4) (layers "F.Cu" "B.Cu") (free) (net 6))
+  (via (at 185.42 86.36) (size 0.8) (drill 0.4) (layers "F.Cu" "B.Cu") (free) (net 6))
   (via (at 142.24 71.12) (size 0.8) (drill 0.4) (layers "F.Cu" "B.Cu") (free) (net 6))
   (via (at 149.86 83.82) (size 0.8) (drill 0.4) (layers "F.Cu" "B.Cu") (free) (net 6))
+  (via (at 185.42 81.28) (size 0.8) (drill 0.4) (layers "F.Cu" "B.Cu") (free) (net 6))
   (via (at 137.16 78.74) (size 0.8) (drill 0.4) (layers "F.Cu" "B.Cu") (free) (net 6))
   (via (at 141.607417 82.767012) (size 0.8) (drill 0.4) (layers "F.Cu" "B.Cu") (free) (net 6))
@@
   (via (at 177.8 78.74) (size 0.8) (drill 0.4) (layers "F.Cu" "B.Cu") (free) (net 6))
   (via (at 99.06 88.9) (size 0.8) (drill 0.4) (layers "F.Cu" "B.Cu") (free) (net 6))
+  (via (at 185.42 76.2) (size 0.8) (drill 0.4) (layers "F.Cu" "B.Cu") (free) (net 6))
   (via (at 149.86 91.44) (size 0.8) (drill 0.4) (layers "F.Cu" "B.Cu") (free) (net 6))
   (via (at 96.52 104.14) (size 0.8) (drill 0.4) (layers "F.Cu" "B.Cu") (free) (net 6))
@@
   (via (at 99.06 91.44) (size 0.8) (drill 0.4) (layers "F.Cu" "B.Cu") (free) (net 6))
   (via (at 93.98 81.28) (size 0.8) (drill 0.4) (layers "F.Cu" "B.Cu") (free) (net 6))
+  (via (at 185.42 114.3) (size 0.8) (drill 0.4) (layers "F.Cu" "B.Cu") (free) (net 6))
   (via (at 93.98 106.68) (size 0.8) (drill 0.4) (layers "F.Cu" "B.Cu") (free) (net 6))
   (via (at 180.34 116.84) (size 0.8) (drill 0.4) (layers "F.Cu" "B.Cu") (free) (net 6))
+  (via (at 147.32 93.98) (size 0.8) (drill 0.4) (layers "F.Cu" "B.Cu") (free) (net 6))
   (via (at 114.3 81.28) (size 0.8) (drill 0.4) (layers "F.Cu" "B.Cu") (free) (net 6))
   (via (at 104.214189 120.323718) (size 0.8) (drill 0.4) (layers "F.Cu" "B.Cu") (free) (net 6))
@@
   (via (at 106.68 81.28) (size 0.8) (drill 0.4) (layers "F.Cu" "B.Cu") (free) (net 6))
   (via (at 160.02 96.52) (size 0.8) (drill 0.4) (layers "F.Cu" "B.Cu") (free) (net 6))
+  (via (at 185.42 119.38) (size 0.8) (drill 0.4) (layers "F.Cu" "B.Cu") (free) (net 6))
   (segment (start 124.732707 123.810239) (end 124.732707 128.86358) (width 0.8) (layer "B.Cu") (net 6))
   (segment (start 124.325606 123.403138) (end 124.732707 123.810239) (width 0.8) (layer "B.Cu") (net 6))
@@
   (segment (start 100.056667 97.42234) (end 100.056667 104.448781) (width 0.25) (layer "F.Cu") (net 18))
   (segment (start 103.029067 96.52234) (end 121.276667 96.52234) (width 0.25) (layer "F.Cu") (net 18))
-  (segment (start 129.86399 113.11185) (end 129.86399 113.157508) (width 0.25) (layer "F.Cu") (net 18))
   (segment (start 103.757246 108.14936) (end 124.9015 108.14936) (width 0.25) (layer "F.Cu") (net 18))
   (via (at 129.86399 113.157508) (size 0.8) (drill 0.4) (layers "F.Cu" "B.Cu") (net 18))
