File: ykp74/ykp74.kicad_sch (KiCad schematic)
At the start: 22 parts, among them U1 27C256, U2 27C256, U3 27C256, U4 27C256, U5 74LS139, U6 74LS32, U7 74LS04, U8 74LS670

Commit message: Change the Foot Print of Edge slot
Signed-off-by: Youngki Park <ykp7409@gmail.com>
Parts:
- removed CE1: Card_Edge_Connector_MSX, ykp74_work_Library:card_edge_connector_MSX, symbol ykp74_work:Card_Edge_Connector_MSX
- added CE1: Card_Edge_Connector_MSX, Lib_add:card_edge_connector_MSX, symbol card_edge_connector_msx:Card_Edge_Connector_MSX
Connections:
- net +5V: now also CE1.45 (+5V), CE1.47 (+5V)
- net A0: now also CE1.28 (A0)
- net A1: now also CE1.27 (A1)
- net A10: now also CE1.20 (A10)
- net A11: now also CE1.19 (A11)
- net A12: now also CE1.23 (A12)
- net A13: now also CE1.26 (A13)
- net A15: now also CE1.18 (A15)
- net A2: now also CE1.30 (A2)
- net A3: now also CE1.29 (A3)
- net A4: now also CE1.32 (A4)
- net A5: now also CE1.31 (A5)
- net A6: now also CE1.22 (A6)
- net A7: now also CE1.21 (A7)
- net A8: now also CE1.24 (A8)
- net A9: now also CE1.17 (A9)
- net D0: now also CE1.34 (D0)
- net D1: now also CE1.33 (D1)
- net D2: now also CE1.36 (D2)
- net D3: now also CE1.35 (D3)
- net D4: now also CE1.38 (D4)
- net D5: now also CE1.37 (D5)
- net D6: now also CE1.40 (D6)
- net D7: now also CE1.39 (D7)
- net GND: now also CE1.41 (GND), CE1.43 (GND)
- net /RD: now also CE1.14 (~{RD})
- net /SLTSL: now also CE1.4 (~{STLSL})
- net /WR: now also CE1.13 (~{WR})
Changed lines of the file:
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@@
+    )
+  )
+  (symbol (lib_id "card_edge_connector_msx:Card_Edge_Connector_MSX") (at 224.79 62.23 0) (unit 1)
+    (in_bom yes) (on_board yes) (dnp no) (fields_autoplaced)
+    (property "Reference" "CE1" (at 224.79 40.64 0)
+      (effects (font (size 1.27 1.27)))
+    )
+    (property "Value" "Card_Edge_Connector_MSX" (at 224.79 43.18 0)
+      (effects (font (size 1.27 1.27)))
+    )
+    (property "Footprint" "Lib_add:card_edge_connector_MSX" (at 224.79 80.01 0)
+      (effects (font (size 1.27 1.27)) hide)
+    )
+    (property "Datasheet" "" (at 224.79 60.96 90)
+      (effects (font (size 1.27 1.27)) hide)
+    )
+    (pin "1")
+    (pin "10")
+    (pin "11")
+    (pin "12")
+    (pin "13")
+    (pin "14")
+    (pin "15")
+    (pin "16")
+    (pin "17")
+    (pin "18")
+    (pin "19")
+    (pin "2")
+    (pin "20")
+    (pin "21")
+    (pin "22")
+    (pin "23")
+    (pin "24")
+    (pin "25")
+    (pin "26")
+    (pin "27")
+    (pin "28")
+    (pin "29")
+    (pin "3")
+    (pin "30")
+    (pin "31")
+    (pin "32")
+    (pin "33")
+    (pin "34")
+    (pin "35")
+    (pin "36")
+    (pin "37")
+    (pin "38")
+    (pin "39")
+    (pin "4")
+    (pin "40")
+    (pin "41")
+    (pin "42")
+    (pin "43")
+    (pin "44")
+    (pin "45")
+    (pin "46")
+    (pin "47")
+    (pin "48")
+    (pin "49")
+    (pin "5")
+    (pin "50")
+    (pin "6")
+    (pin "7")
+    (pin "8")
+    (pin "9")
+    (instances
+      (project "ykp74"
+        (path "/24ee4311-09c0-43df-93e6-94a6fb22b16b"
+          (reference "CE1") (unit 1)
+        )
+      )
     )
   )
@@
         )
       )
-    )
-  )
-  (symbol (lib_id "ykp74_work:Card_Edge_Connector_MSX") (at 224.79 62.23 0) (unit 1)
-    (in_bom yes) (on_board yes) (dnp no) (fields_autoplaced)
-    (property "Reference" "CE1" (at 224.79 40.64 0)
-      (effects (font (size 1.27 1.27)))
-    )
-    (property "Value" "Card_Edge_Connector_MSX" (at 224.79 43.18 0)
-      (effects (font (size 1.27 1.27)))
-    )
-    (property "Footprint" "ykp74_work_Library:card_edge_connector_MSX" (at 226.06 78.74 0)
-      (effects (font (size 1.27 1.27)))
-    )
-    (property "Datasheet" "" (at 224.79 60.96 90)
-      (effects (font (size 1.27 1.27)) hide)
-    )
-    (pin "1")
-    (pin "10")
-    (pin "11")
-    (pin "12")
-    (pin "13")
-    (pin "14")
-    (pin "15")
-    (pin "16")
-    (pin "17")
-    (pin "18")
-    (pin "19")
-    (pin "2")
-    (pin "20")
-    (pin "21")
-    (pin "22")
-    (pin "23")
-    (pin "24")
-    (pin "25")
-    (pin "26")
-    (pin "27")
-    (pin "28")
-    (pin "29")
-    (pin "3")
-    (pin "30")
-    (pin "31")
-    (pin "32")
-    (pin "33")
-    (pin "34")
-    (pin "35")
-    (pin "36")
-    (pin "37")
-    (pin "38")
-    (pin "39")
-    (pin "4")
-    (pin "40")
-    (pin "41")
-    (pin "42")
-    (pin "43")
-    (pin "44")
-    (pin "45")
-    (pin "46")
-    (pin "47")
-    (pin "48")
-    (pin "49")
-    (pin "5")
-    (pin "50")
-    (pin "6")
-    (pin "7")
-    (pin "8")
-    (pin "9")
-    (instances
-      (project "ykp74"
-        (path "/24ee4311-09c0-43df-93e6-94a6fb22b16b"
-          (reference "CE1") (unit 1)
-        )
-      )
