File: project4/project4.kicad_pcb (KiCad board)
At the start: 2 copper layers, 100.8 x 98.2 mm, 33 parts, among them J1 Conn_02x03, J2 Conn_02x03, J3 Conn_02x03, J4 Conn_02x03, J5 Conn_02x03, J6 Conn_02x02, U1 SST27ST020, U2 SST27ST020, U3 SST27ST020, U4 SST27ST020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

Commit message: Added new project2-2
Signed-off-by: Youngki Park <ykp7409@gmail.com>
Parts:
- moved C1 0.63 mm to (125.7, 89.5)
- moved C2 0.63 mm to (146.0, 89.5)
- moved C3 0.63 mm to (166.3, 89.5)
- moved C4 0.63 mm to (186.6, 89.5)
Routing:
- net +5V: track 422.0 -> 418.4 mm, vias 1 -> 2
- net GND: vias 132 -> 106
