File: project2_2/project2_2.kicad_sch (KiCad schematic)
At the start: 28 parts, among them J1 Conn_02x02, J5 Conn_02x02, U1 AT27C020, U2 AT27C020, U3 74LS32, U5 74LS670, U8 74LS00

Commit message: modify PCB 2-2
Signed-off-by: Youngki Park <ykp7409@gmail.com>
Parts:
- removed CE?: Card_Edge_Connector_MSX, Lib_add:card_edge_connector_MSX, symbol ykp74_work:Card_Edge_Connector_MSX
- removed J1: Conn_02x02, symbol Connector_Generic:Conn_02x02_Odd_Even
- added CE1: Card_Edge_Connector_MSX, Lib_add:card_edge_connector_MSX, symbol card_edge_connector_msx:Card_Edge_Connector_MSX
- added J2: Conn_02x03, Connector_PinHeader_2.54mm:PinHeader_2x03_P2.54mm_Vertical, symbol Connector_Generic:Conn_02x03_Odd_Even
- added J3, J4: Conn_02x02, Connector_PinHeader_2.54mm:PinHeader_2x02_P2.54mm_Vertical, symbol Connector_Generic:Conn_02x02_Odd_Even
- C? (x7): value 100n -> 0.1uF
- C?: value 10uf -> 10uF
- J1: renamed from J5; footprint (none) -> Connector_PinHeader_2.54mm:PinHeader_2x02_P2.54mm_Vertical
- R? (x6): value 470R -> 470
- U5: renamed from U3; footprint (none) -> Package_DIP:DIP-14_W7.62mm_Socket
- U6: renamed from U8; footprint (none) -> Package_DIP:DIP-14_W7.62mm_Socket
- U?: renamed from U5; footprint (none) -> Package_DIP:DIP-16_W7.62mm_Socket
Connections:
- net /Er is gone; now on net GND: U?.11 (~{Er}), U?.11 (~{Er})
- net +5V: now also CE1.45 (+5V), CE1.47 (+5V)
- net A0: now also CE1.28 (A0)
- net A1: now also CE1.27 (A1)
- net A10: now also CE1.20 (A10)
- net A11: now also CE1.19 (A11), J2.1 (Pin_1)
- net A12: now also CE1.23 (A12), J2.3 (Pin_3)
- net A13: now also U1.28 (A13), U2.28 (A13), CE1.26 (A13); no longer U?.4 (Rb), U?.4 (Rb)
- net A14: now also CE1.25 (A14)
- net A15: now also CE1.18 (A15), J3.1 (Pin_1), J4.3 (Pin_3); no longer U?.5 (Ra), U?.5 (Ra)
- net A2: now also CE1.30 (A2)
- net A3: now also CE1.29 (A3)
- net A4: now also CE1.32 (A4)
- net A5: now also CE1.31 (A5)
- net A6: now also CE1.22 (A6)
- net A7: now also CE1.21 (A7)
- net A8: now also CE1.24 (A8)
- net A9: now also CE1.17 (A9)
- net D0: now also U?.15 (D1), CE1.34 (D0); no longer U?.3 (D4)
- net D1: now also U?.1 (D2), CE1.33 (D1); no longer U?.2 (D3)
- net D2: now also U?.2 (D3), CE1.36 (D2); no longer U?.1 (D2)
- net D3: now also U?.3 (D4), CE1.35 (D3); no longer U?.15 (D1)
- net D4: now also CE1.38 (D4)
- net D5: now also CE1.37 (D5)
- net D6: now also CE1.40 (D6)
- net D7: now also CE1.39 (D7)
- net GND: now also CE1.41 (GND), CE1.43 (GND), J2.5 (Pin_5), J3.3 (Pin_3), J4.1 (Pin_1); no longer U?.3 (A1)
- net MA14: now also R?.2, U?.10 (Q1); no longer R?.2, U?.7 (Q3)
- net MA16: now also R?.2, U?.7 (Q3); no longer R?.2, U?.10 (Q1)
- net MA17: now also R?.2, U?.6 (Q4); no longer R?.2, U?.10 (Q1)
- net /RD: now also CE1.14 (~{RD})
- net /SLTSL: now also CE1.4 (~{STLSL})
- net /WR: now also CE1.13 (~{WR})
- net at U?.13 (Wb), U?.13 (Wb): now also J2.2 (Pin_2), J2.4 (Pin_4), J2.6 (Pin_6)
- net at R?.2, U?.9 (Q2): now also U?.3 (A1); no longer U?.2 (A0)
- removed net MA13: R?.2, U1.28 (A13), U2.28 (A13), U?.6 (Q4)
- new net: R?.2, U?.10 (Q1), U?.2 (A0)
- new net: J3.2 (Pin_2), J3.4 (Pin_4), U?.5 (Ra), U?.5 (Ra)
- new net: J4.2 (Pin_2), J4.4 (Pin_4), U?.4 (Rb), U?.4 (Rb)
- no-connect marks 26 -> 37
Other:
- moved on the sheet: C?, J1, U?A

Commit message: Final revision
Signed-off-by: Youngki Park <ykp7409@gmail.com>
Connections:
- net GND: now also U?.2 (D3), U?.3 (D4)
- no-connect marks 37 -> 33
Other:
- moved on the sheet: U?A
Changed lines of the file:
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@@
 (kicad_sch (version 20230121) (generator eeschema)
   (paper "A4")
+  (title_block
+    (date "2023-06-02")
+    (rev "1.2")
+  )
   (junction (at 121.92 115.57) (diameter 0) (color 0 0 0 0)
   )
@@
   (junction (at 38.1 87.63) (diameter 0) (color 0 0 0 0)
   )
+  (junction (at 87.63 123.19) (diameter 0) (color 0 0 0 0)
+  )
   (junction (at 204.47 83.82) (diameter 0) (color 0 0 0 0)
   )
@@
   (no_connect (at 228.6 21.59))
   (no_connect (at 228.6 46.99))
-  (no_connect (at 165.1 120.65))
   (no_connect (at 238.76 48.26))
   (no_connect (at 238.76 20.32))
@@
   (no_connect (at 15.24 129.54))
   (no_connect (at 228.6 20.32))
+  (no_connect (at 33.02 138.43))
   (no_connect (at 228.6 26.67))
   (no_connect (at 30.48 127))
   (no_connect (at 31.75 124.46))
-  (no_connect (at 91.44 120.65))
   (no_connect (at 228.6 24.13))
   (no_connect (at 30.48 142.24))
   (no_connect (at 48.26 140.97))
   (no_connect (at 238.76 24.13))
-  (no_connect (at 91.44 123.19))
-  (no_connect (at 33.02 138.43))
-  (no_connect (at 165.1 118.11))
   (no_connect (at 238.76 21.59))
   (no_connect (at 46.99 127))
@@
     (stroke (width 0) (type default))
   )
+  (wire (pts (xy 91.44 120.65) (xy 87.63 120.65))
+    (stroke (width 0) (type default))
+  )
   (wire (pts (xy 231.14 137.16) (xy 236.22 137.16))
     (stroke (width 0) (type default))
@@
     (stroke (width 0) (type default))
   )
-  (wire (pts (xy 121.92 115.57) (xy 139.7 115.57))
+  (wire (pts (xy 121.92 115.57) (xy 133.35 115.57))
     (stroke (width 0) (type default))
   )
@@
     (stroke (width 0) (type default))
   )
+  (wire (pts (xy 87.63 120.65) (xy 87.63 123.19))
+    (stroke (width 0) (type default))
+  )
   (wire (pts (xy 231.14 129.54) (xy 236.22 129.54))
     (stroke (width 0) (type default))
@@
     (stroke (width 0) (type default))
   )
+  (wire (pts (xy 158.75 118.11) (xy 162.56 118.11))
+    (stroke (width 0) (type default))
+  )
   (wire (pts (xy 228.6 139.7) (xy 228.6 142.24))
     (stroke (width 0) (type default))
@@
     (stroke (width 0) (type default))
   )
-  (wire (pts (xy 134.62 120.65) (xy 139.7 120.65))
-    (stroke (width 0) (type default))
-  )
   (wire (pts (xy 22.86 69.85) (xy 25.4 69.85))
     (stroke (width 0) (type default))
@@
     (stroke (width 0) (type default))
   )
-  (wire (pts (xy 139.7 113.03) (xy 132.08 113.03))
-    (stroke (width 0) (type default))
-  )
   (wire (pts (xy 243.84 31.75) (xy 238.76 31.75))
     (stroke (width 0) (type default))
@@
     (stroke (width 0) (type default))
   )
-  (wire (pts (xy 119.38 118.11) (xy 132.08 118.11))
+  (wire (pts (xy 119.38 118.11) (xy 133.35 118.11))
     (stroke (width 0) (type default))
   )
@@
     (stroke (width 0) (type default))
   )
+  (wire (pts (xy 87.63 123.19) (xy 91.44 123.19))
+    (stroke (width 0) (type default))
+  )
   (wire (pts (xy 69.85 143.51) (xy 91.44 143.51))
     (stroke (width 0) (type default))
@@
     (stroke (width 0) (type default))
   )
-  (wire (pts (xy 165.1 113.03) (xy 168.91 113.03))
+  (wire (pts (xy 125.73 110.49) (xy 133.35 110.49))
     (stroke (width 0) (type default))
   )
@@
     (stroke (width 0) (type default))
   )
-  (wire (pts (xy 165.1 115.57) (xy 168.91 115.57))
+  (wire (pts (xy 158.75 115.57) (xy 162.56 115.57))
     (stroke (width 0) (type default))
   )
@@
     (stroke (width 0) (type default))
   )
+  (wire (pts (xy 87.63 123.19) (xy 87.63 124.46))
+    (stroke (width 0) (type default))
+  )
   (wire (pts (xy 87.63 67.31) (xy 91.44 67.31))
     (stroke (width 0) (type default))
@@
     (stroke (width 0) (type default))
   )
-  (wire (pts (xy 132.08 118.11) (xy 132.08 113.03))
-    (stroke (width 0) (type default))
-  )
   (wire (pts (xy 256.54 106.68) (xy 259.08 106.68))
     (stroke (width 0) (type default))
@@
     (effects (font (size 1.27 1.27)) (justify left bottom))
   )
-  (label "ROM_CE2" (at 168.91 115.57 0) (fields_autoplaced)
+  (label "ROM_CE2" (at 162.56 115.57 0) (fields_autoplaced)
     (effects (font (size 1.27 1.27)) (justify left bottom))
   )
@@
     (effects (font (size 1.27 1.27)) (justify left bottom))
   )
+  (label "{slash}SLTSL" (at 125.73 110.49 0) (fields_autoplaced)
+    (effects (font (size 1.27 1.27)) (justify left bottom))
+  )
   (label "A5" (at 232.41 106.68 0) (fields_autoplaced)
     (effects (font (size 1.27 1.27)) (justify left bottom))
@@
     (effects (font (size 0.7 0.7)) (justify left bottom))
   )
-  (label "ROM_CE1" (at 168.91 113.03 0) (fields_autoplaced)
+  (label "ROM_CE1" (at 162.56 118.11 0) (fields_autoplaced)
     (effects (font (size 1.27 1.27)) (justify left bottom))
   )
@@
     (effects (font (size 0.7 0.7)) (justify left bottom))
   )
-  (label "{slash}SLTSL" (at 134.62 120.65 0) (fields_autoplaced)
-    (effects (font (size 1.27 1.27)) (justify left bottom))
-  )
   (label "D2" (at 217.17 99.06 0) (fields_autoplaced)
     (effects (font (size 1.27 1.27)) (justify left bottom))
@@
     )
   )
+  (symbol (lib_id "power:GND") (at 87.63 124.46 0) (unit 1)
+    (in_bom yes) (on_board yes) (dnp no) (fields_autoplaced)
+    (property "Reference" "#PWR036" (at 87.63 130.81 0)
+      (effects (font (size 1.27 1.27)) hide)
+    )
+    (property "Value" "GND" (at 87.63 129.54 0)
+      (effects (font (size 1.27 1.27)))
+    )
+    (property "Footprint" "" (at 87.63 124.46 0)
+      (effects (font (size 1.27 1.27)) hide)
+    )
+    (property "Datasheet" "" (at 87.63 124.46 0)
+      (effects (font (size 1.27 1.27)) hide)
+    )
+    (pin "1")
+    (instances
+      (project "project2_2"
+        (path "/39de7e4e-14d0-48bf-9a69-30d0c1286532"
+          (reference "#PWR036") (unit 1)
+        )
+      )
+    )
+  )
   (symbol (lib_id "Connector_Generic:Conn_02x02_Odd_Even") (at 30.48 58.42 0) (unit 1)
     (in_bom yes) (on_board yes) (dnp no) (fields_autoplaced)
@@
     )
   )
-  (symbol (lib_id "74xx:74LS139") (at 152.4 115.57 0) (unit 1)
-    (in_bom yes) (on_board yes) (dnp no) (fields_autoplaced)
-    (property "Reference" "U?" (at 152.4 106.68 0)
+  (symbol (lib_id "74xx:74LS139") (at 146.05 115.57 0) (mirror x) (unit 1)
+    (in_bom yes) (on_board yes) (dnp no)
+    (property "Reference" "U?" (at 146.05 124.46 0)
       (effects (font (size 1.27 1.27)))
     )
-    (property "Value" "74LS139" (at 152.4 109.22 0)
+    (property "Value" "74LS139" (at 146.05 121.92 0)
       (effects (font (size 1.27 1.27)))
     )
-    (property "Footprint" "Package_DIP:DIP-16_W7.62mm_Socket" (at 152.4 115.57 0)
+    (property "Footprint" "Package_DIP:DIP-16_W7.62mm_Socket" (at 146.05 115.57 0)
       (effects (font (size 1.27 1.27)) hide)
     )
-    (property "Datasheet" "http://www.ti.com/lit/ds/symlink/sn74ls139a.pdf" (at 152.4 115.57 0)
+    (property "Datasheet" "http://www.ti.com/lit/ds/symlink/sn74ls139a.pdf" (at 146.05 115.57 0)
       (effects (font (size 1.27 1.27)) hide)
     )
