File: project_memory_mapper/project_memory_mapper.kicad_pcb (KiCad board)
At the start: 2 copper layers, 18 parts, among them U1 74LS30, U2 74LS139, U3 74LS670, U4 74LS670, U5 CS18LV10245, U6 CS18LV10245, U7 CS18LV10245, U8 CS18LV10245

Commit message: modify pcb
Signed-off-by: ykp74 <ykp7409@gmail.com>
Routing:
- net Net-(U2B-O0): track 67.6 -> 68.3 mm
- net /D4: track 172.2 -> 172.9 mm
- net +5V: track 339.1 -> 339.7 mm
- net GND: vias 0 -> 50
- added copper zone on B.Cu, net GND
- added copper zone on F.Cu, net GND
Other:
- board outline added: 100.7 x 77.2 mm

Commit message: modified PCB : Signed-off-by: ykp74 <ykp7409@gmail.com>
Parts:
- moved C3 1.23 mm to (102.9, 45.5)
Routing:
- net /A0: track 173.9 -> 172.8 mm
- net Net-(U2B-O0): track 68.3 -> 67.6 mm
- net /A1: track 175.7 -> 176.2 mm
- net /D0: track 142.2 -> 141.7 mm
- net GND: vias 50 -> 56

Commit message: PCB Released
Signed-off-by: Youngki Park <ykp7409@gmail.com>
Other:
- board text added: "Expansion Memory 1.0 Designed By ykp74"
